File: ArcadeKicad/ArcadeKicad.kicad_sch (KiCad schematic)
At the start: 18 parts, among them J2 TVout, J3 joystick, J4 Bornera, SW1 SW_Push, U1 ATMEGA328P-PU, U2 L7805, Y1 Crystal_Small

Commit message: PCB
primer diseño de pcb
Parts:
- C1, C2: footprint (none) -> Capacitor_SMD:C_1210_3225Metric_Pad1.33x2.70mm_HandSolder
- C3, C4: footprint EESTN5:CAP_ELEC_8x11.5mm -> Capacitor_SMD:C_1210_3225Metric_Pad1.33x2.70mm_HandSolder
- D1: footprint (none) -> LED_SMD:LED_1210_3225Metric
- J3: footprint Connector_Hirose:Hirose_DF13-05P-1.25DSA_1x05_P1.25mm_Vertical -> EESTN5:Pin_Strip_5
- R1, R2, R3: footprint (none) -> EESTN5:R_1206
- R4: footprint Resistor_THT:R_Axial_DIN0204_L3.6mm_D1.6mm_P5.08mm_Horizontal -> EESTN5:R_1206
- SW1: footprint (none) -> EESTN5:SW_SPST_EVQPE1
- TP1, TP2: footprint TestPoint:TestPoint_Loop_D2.50mm_Drill1.0mm_LowProfile -> TestPoint:TestPoint_Keystone_5015_Micro-Minature
- U2: footprint EESTN5:TO-220 -> Package_TO_SOT_SMD:TSOT-23_HandSoldering
Connections:
- net +5V is gone; now on net +5v: C4.1, TP1.1, U2.3 (OUT)
- net Xjoy: now also U1.23 ((PCINT8/ADC0)PC0)
- net Yjoy: now also U1.24 ((PCINT9/ADC1)PC1)
- net pulsador: now also U1.17 ((PCINT3/OC2A/MOSI)PB3)
- net Led: now reaches D1.2 (A), U1.19 ((PCINT5/SCK)PB5)
- net Reset: now reaches SW1.1, U1.1 ((PCINT14/~{RESET})PC6)
Other:
- note added: "ATmega"
- note added: "Joystick"
- note added: "conexiones TVout"
- moved on the sheet: C1, C2, C3, C4, D1, J4, R1, R2, SW1, TP1, TP2, U1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
